File: hardware/output/machine-room-monitor-schematic.kicad_sch (KiCad schematic)
At the start: 20 parts, among them J1 USB-TTL (CH340), J2 ST-Link V2 (SWD), SW1 RESET, U1 STM32F103C8T6, U2 DHT11, U3 MQ-2, U4 BH1750, Y1 8MHz

Commit message: 文档与命名规范化：统一模块命名与表述
- 模块命名统一为 单片机端 / 客户端 / 服务器端，去掉早期的任务编号前缀
- 文档重命名（保留 git 历史）：任务A-单片机端.md → 单片机端.md 等 6 个文档
- 原理图文件名 taskA → schematic，标题与图签栏重新导出（Proteus / kicad-cli）
- 代码注释、脚本、SQL、模拟器说明同步更新
- 技术术语保持不变（线程池"任务队列"、"规划 S5 任务 N"条目引用等）
Other:
- title: 机房环境监测系统 · 任务A 单片机端原理图 -> 机房环境监测系统 · 单片机端原理图
Changed lines of the file:
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@@
 	(paper "A3")
 	(title_block
-		(title "机房环境监测系统 · 任务A 单片机端原理图")
+		(title "机房环境监测系统 · 单片机端原理图")
 		(date "2026-10-09")
 		(rev "A")
